File: Animatronics 12v to 5V Converter/4x board.brd (EAGLE design)
At the start: 87.9 x 67.1 mm, 27 parts, among them J1 1017504, J2 1017504, J3 1017504, J4 1017504, J5 2606-3102/020-000, U1 MC7805CTG, U2 MC7805CTG, U3 MC7805CTG, U4 MC7805CTG

Commit message: Finished PCB
Parts:
- removed J1, J2, J3, J4: 1017504, 1017504:1017504
- added IN1, IN2, IN3, IN4: WEIDMUELLER_1825970000WEIDMUELLER_1825970000_0_0, Weidmueller - 1825970000:WEIDMUELLER_1825970000_0
Connections:
- new net N$11: R1.5, R2.5, U4.3
- net +12V: now also IN1.A2, IN1.A2-2, IN2.A2, IN2.A2-2, IN3.A2, IN3.A2-2, IN4.A2, IN4.A2-2; no longer J1.5, J1.6, J2.5, J2.6, J3.5, J3.6, J4.5, J4.6
- net GND: now also IN1.A3, IN1.A3-2, IN2.A3, IN2.A3-2, IN3.A3, IN3.A3-2, IN4.A3, IN4.A3-2; no longer J1.3, J1.4, J2.3, J2.4, J3.3, J3.4, J4.3, J4.4
- net N$2: now also IN2.A1, IN2.A1-2; no longer J1.1, J1.2
- net N$23: now also IN1.A1, IN1.A1-2; no longer J2.1, J2.2
- net N$5: no longer R1.5, R2.5, U4.3
- net N$6: now also IN3.A1, IN3.A1-2; no longer J3.1, J3.2
- net N$8: now also IN4.A1, IN4.A1-2; no longer J4.1, J4.2
Routing:
- net GND: track 0.00 -> 253.3 mm
- net +12V: track 0.00 -> 123.6 mm
- net N$5: track 0.00 -> 111.9 mm
- net N$11: track 0.00 -> 104.4 mm, vias 0 -> 1
- net N$9: track 0.00 -> 98.7 mm
- net N$10: track 0.00 -> 90.4 mm, vias 0 -> 1
- net N$7: track 0.00 -> 72.0 mm
- net N$20: track 0.00 -> 66.2 mm, vias 0 -> 1
- net N$3: track 0.00 -> 57.9 mm
- net N$23: track 0.00 -> 45.9 mm
- net N$17: track 0.00 -> 44.7 mm, vias 0 -> 1
- net N$1: track 0.00 -> 44.2 mm
- net N$4: track 0.00 -> 42.8 mm
- net N$19: track 0.00 -> 33.3 mm
- net N$2: track 0.00 -> 29.2 mm
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Other:
- board size 87.9 x 67.1 mm -> 87.9 x 58.2 mm
- board text added: "Designed By Nate; 2022"
- board text added: "For The Original EAGLE Files Go To: https://github.com/Moving-Light/PCbs"
- board text added: "JLCJLCJLCJLC"
