File: Animatronics 12v to 5V Converter/4x board.sch (EAGLE design)
At the start: 27 parts, among them J1 1017504, J2 1017504, J3 1017504, J4 1017504, J5 2606-3102/020-000, U1 MC7805CTG, U2 MC7805CTG, U3 MC7805CTG, U4 MC7805CTG

Commit message: Finished PCB
Parts:
- removed J1, J2, J3, J4: 1017504, 1017504:1017504
- added IN1, IN2, IN3, IN4: WEIDMUELLER_1825970000WEIDMUELLER_1825970000_0_0, Weidmueller - 1825970000:WEIDMUELLER_1825970000WEIDMUELLER_1825970000_0_0
Connections:
- new net N$11: R1.5, R2.5, U4.OUTPUT
- net +12V: now also IN1B.A2, IN2B.A2, IN3B.A2, IN4B.A2; no longer J1.3.1, J1.3.2, J2.3.1, J2.3.2, J3.3.1, J3.3.2, J4.3.1, J4.3.2
- net GND: now also IN1C.A3, IN2C.A3, IN3C.A3, IN4C.A3; no longer J1.2.1, J1.2.2, J2.2.1, J2.2.2, J3.2.1, J3.2.2, J4.2.1, J4.2.2
- net N$2: now also IN2A.A1; no longer J1.1.1, J1.1.2
- net N$23: now also IN1A.A1; no longer J2.1.1, J2.1.2
- net N$5: no longer R1.5, R2.5, U4.OUTPUT
- net N$6: now also IN3A.A1; no longer J3.1.1, J3.1.2
- net N$8: now also IN4A.A1; no longer J4.1.1, J4.1.2
